File: aeronode.kicad_pcb (KiCad board)
At the start: 2 copper layers, 60 x 60 mm, 9 parts, among them J1 Conn_01x08

Commit message: backup commit
Parts:
- removed ELRS1, FC1, SERIAL1: Conn_01x04_Socket, Connector_PinSocket_2.54mm:PinSocket_1x04_P2.54mm_Vertical
- removed G***: LOGO, LOGO
- removed J1: Conn_01x08, Connector_PinSocket_2.54mm:PinSocket_1x08_P2.54mm_Vertical
- removed MUX1: Conn_02x08_Counter_Clockwise, Connector_PinHeader_2.54mm:PinHeader_2x8_2.54mm_7.62mm
- removed SignalConverter1: Conn_02x06_Counter_Clockwise, Connector_PinHeader_2.54mm:PinHeader_2x6_2.54mm_10.16mm
- removed U1, U2: ~, pico_2:PICO2-SMD
Routing:
- net GND: track 336.9 -> 0.00 mm, vias 2 -> 0
- net +3V3: track 89.2 -> 0.00 mm, vias 5 -> 0
- net Net-(MUX1-Pin_13): track 83.8 -> 0.00 mm, vias 1 -> 0
- net Net-(MUX1-Pin_14): track 48.9 -> 0.00 mm
- net Net-(SERIAL1-Pin_2): track 42.9 -> 0.00 mm
- net Net-(SERIAL1-Pin_3): track 40.0 -> 0.00 mm
- net Net-(MUX1-Pin_11): track 30.0 -> 0.00 mm
- net Net-(ELRS1-Pin_3): track 29.9 -> 0.00 mm, vias 1 -> 0
- net Net-(J1-Pin_8): track 28.4 -> 0.00 mm, vias 2 -> 0
- net Net-(J1-Pin_7): track 26.9 -> 0.00 mm, vias 2 -> 0
- net +5V: track 23.6 -> 0.00 mm
- net Net-(MUX1-Pin_3): track 22.1 -> 0.00 mm
- net Net-(U1-GP22): track 19.6 -> 0.00 mm, vias 1 -> 0
- net Net-(U1-GP26): track 19.5 -> 0.00 mm, vias 1 -> 0
- net Net-(J1-Pin_5): track 18.4 -> 0.00 mm
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- removed copper zone on B.Cu, net GND
- removed copper zone on F.Cu, net GND
Other:
- board outline removed
- board text removed: "AeroNode v0"

Commit message: v0.1
Parts:
- added C1: 22u, Capacitor_SMD:C_0805_2012Metric, F.Cu at (85.6, 96.4)
- added C10: 2u2, Capacitor_SMD:C_0402_1005Metric, F.Cu at (102.3, 88.5)
- added C11: 100n, Capacitor_SMD:C_0402_1005Metric, F.Cu at (108.3, 103.5)
- added C12: 100n, Capacitor_SMD:C_0402_1005Metric, F.Cu at (100.8, 88.9)
- added C13: 100n, Capacitor_SMD:C_0402_1005Metric, F.Cu at (96.6, 91.9)
- added C14: 100n, Capacitor_SMD:C_0402_1005Metric, F.Cu at (101.4, 103.5)
- added C15: 1u, Capacitor_SMD:C_0402_1005Metric, F.Cu at (96.9, 98.3)
- added C16: 100n, Capacitor_SMD:C_0402_1005Metric, F.Cu at (95.8, 98.3)
- added C17: 1u, Capacitor_SMD:C_0402_1005Metric, F.Cu at (94.7, 98.3)
- added C18: 100n, Capacitor_SMD:C_0402_1005Metric, B.Cu at (106.1, 83.7)
- added C19: 10u, Capacitor_SMD:C_0402_1005Metric, B.Cu at (99.2, 89.7)
- added C2: 100n, Capacitor_SMD:C_0402_1005Metric, F.Cu at (92.9, 102.7)
- added C20: 100n, Capacitor_SMD:C_0402_1005Metric, B.Cu at (112.6, 95.0)
- added C21: 100n, Capacitor_SMD:C_0402_1005Metric, B.Cu at (115.3, 93.0)
- added C22: 100n, Capacitor_SMD:C_0402_1005Metric, B.Cu at (103.2, 85.4)
- added C23: 100n, Capacitor_SMD:C_0402_1005Metric, B.Cu at (109.0, 85.8)
- added C24: 100n, Capacitor_SMD:C_0402_1005Metric, B.Cu at (118.0, 95.1)
- added C3: 100n, Capacitor_SMD:C_0402_1005Metric, F.Cu at (92.5, 87.6)
- added C4: 22u, Capacitor_SMD:C_0805_2012Metric, B.Cu at (84.6, 96.8)
- added C5: 10p, Capacitor_SMD:C_0402_1005Metric, F.Cu at (96.8, 93.7)
- added C6: 10p, Capacitor_SMD:C_0402_1005Metric, F.Cu at (96.8, 95.7)
- added C7: 4u7, Capacitor_SMD:C_0603_1608Metric, F.Cu at (101.4, 104.9)
- added C8: 2u2, Capacitor_SMD:C_0402_1005Metric, F.Cu at (106.8, 104.0)
- added C9: 100n, Capacitor_SMD:C_0402_1005Metric, F.Cu at (111.8, 92.6)
- added D1: RED, LED_SMD:LED_0603_1608Metric, F.Cu at (83.6, 80.9)
- added D2: RED, LED_SMD:LED_0603_1608Metric, F.Cu at (83.5, 111.4)
- added FB1: 120R, Inductor_SMD:L_0603_1608Metric, F.Cu at (95.3, 100.1)
- added H1: M4, MountingHole:MountingHole_4.3mm_M4, F.Cu at (89.2, 81.0)
- added H2: M4, MountingHole:MountingHole_4.3mm_M4, F.Cu at (119.7, 81.0)
- added H3: M4, MountingHole:MountingHole_4.3mm_M4, F.Cu at (119.7, 111.5)
- added H4: M4, MountingHole:MountingHole_4.3mm_M4, F.Cu at (89.2, 111.5)
- added J1: FC, Connector_JST:JST_GH_SM04B-GHS-TB_1x04-1MP_P1.25mm_Horizontal, F.Cu at (109.6, 114.7)
- added J2: UART1, Connector_JST:JST_GH_SM04B-GHS-TB_1x04-1MP_P1.25mm_Horizontal, F.Cu at (122.9, 101.4)
- added J3: UART11, Connector_JST:JST_GH_SM04B-GHS-TB_1x04-1MP_P1.25mm_Horizontal, F.Cu at (99.1, 114.7)
- added J4: UART2, Connector_JST:JST_GH_SM04B-GHS-TB_1x04-1MP_P1.25mm_Horizontal, F.Cu at (122.9, 90.8)
- added J5: SWD, Connector_JST:JST_GH_SM04B-GHS-TB_1x04-1MP_P1.25mm_Horizontal, F.Cu at (109.7, 77.7)
- added J6: I2C1, Connector_JST:JST_GH_SM04B-GHS-TB_1x04-1MP_P1.25mm_Horizontal, F.Cu at (99.1, 77.5)
- added J7: Conn_01x01, Connector_Wire:SolderWirePad_1x01_SMD_2x4mm, F.Cu at (85.6, 93.2)
- added J8: Conn_01x01, Connector_Wire:SolderWirePad_1x01_SMD_2x4mm, F.Cu at (85.6, 99.5)
- added Q1: BSS138, PCM_JLCPCB:Q_SOT-23, F.Cu at (109.2, 107.6)
- added Q2: BSS138, PCM_JLCPCB:Q_SOT-23, F.Cu at (113.1, 107.6)
- added R1: 1k5, Resistor_SMD:R_0402_1005Metric, F.Cu at (85.1, 115.6)
- added R2: 1k5, Resistor_SMD:R_0402_1005Metric, F.Cu at (84.5, 76.8)
- added R3: 10k, Resistor_SMD:R_0402_1005Metric, F.Cu at (92.9, 103.9)
- added R4: 10k, Resistor_SMD:R_0402_1005Metric, F.Cu at (93.0, 90.6)
- added R6: 10k, Resistor_SMD:R_0402_1005Metric, F.Cu at (108.8, 105.0)
- added R7: 10k, Resistor_SMD:R_0402_1005Metric, F.Cu at (106.8, 109.2)
- added R8: 10k, Resistor_SMD:R_0402_1005Metric, F.Cu at (113.5, 104.8)
- added R9: 10k, Resistor_SMD:R_0402_1005Metric, F.Cu at (112.8, 110.4)
- added S1: Tactile Button, 160gf, PCM_JLCPCB:SW-SMD_4P-L5.1-W5.1-P3.70-LS6.5-TL-2, F.Cu at (87.3, 88.8)
- added S2: Tactile Button, 160gf, PCM_JLCPCB:SW-SMD_4P-L5.1-W5.1-P3.70-LS6.5-TL-2, F.Cu at (87.4, 103.7)
- added U1: AMS1117-3.3, Package_TO_SOT_SMD:SOT-223-3_TabPin2, B.Cu at (93.0, 96.3)
- added U2: STM32H573RITx, Package_QFP:LQFP-64_10x10mm_P0.5mm, F.Cu at (104.4, 96.2)
- added U3: BMP390, BMP390:10LGA_2X2X0p75_BOS, B.Cu at (99.3, 87.5)
- added U4: ICM-20649, ICM20649:QFN24_3X3X0P9_IVS, B.Cu at (115.3, 95.6)
- added U5: ICM-20649, ICM20649:QFN24_3X3X0P9_IVS, B.Cu at (106.1, 86.3)
- added Y1: 25MHz, Crystal:Crystal_SMD_3225-4Pin_3.2x2.5mm, F.Cu at (92.9, 94.3)
Routing:
- net +3V3: track 0.00 -> 256.2 mm, vias 0 -> 14
- net GND: track 0.00 -> 239.1 mm, vias 0 -> 12
- net I2C1_SCL: track 0.00 -> 52.1 mm, vias 0 -> 2
- net I2C1_SDA: track 0.00 -> 47.6 mm, vias 0 -> 3
- net +5V: track 0.00 -> 46.0 mm, vias 0 -> 3
- net BOOT0: track 0.00 -> 32.2 mm, vias 0 -> 4
- net USART2_TX: track 0.00 -> 27.4 mm, vias 0 -> 2
- net USART2_RX: track 0.00 -> 27.2 mm, vias 0 -> 2
- net NRST: track 0.00 -> 25.2 mm, vias 0 -> 2
- net LED: track 0.00 -> 21.8 mm, vias 0 -> 2
- net SWDIO: track 0.00 -> 15.5 mm
- net FC_TX: track 0.00 -> 13.5 mm
- net USART1_RX: track 0.00 -> 12.8 mm, vias 0 -> 2
- net USART11_RX: track 0.00 -> 12.6 mm
- net USART11_TX: track 0.00 -> 11.9 mm, vias 0 -> 2
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- added copper zone on B.Cu, net GND
- added copper zone on F.Cu, net GND
- added copper zone on In1.Cu, net GND
- added copper zone on In2.Cu, net GND
Other:
- board outline added: 44 x 44 mm
- copper layers 2 -> 4
- board text added: "+"
- board text added: "-"
- board text added: "1"
- board text added: "11"
- board text added: "2"
- board text added: "AeroNode"
- board text added: "BOOT"
- board text added: "CLK"
- board text added: "Designed in San Francisco"
- board text added: "FC"
- board text added: "I2C"
- board text added: "IO"
- board text added: "Moonlit Garage, Inc."
- board text added: "NRST"
- board text added: "R"
- board text added: "SCL"
- board text added: "SDA"
- board text added: "SWD"
- board text added: "T"
- board text added: "v0.1"
